Commit message: rewrite choreo module

File: src/coop_assembly/data/models/kuka_kr6_r900/urdf/mit_arch_grasp_end_effector.urdf (robot description, URDF)
Before this commit: robot mit_arch_grasp_end_effector, 2 links, 1 joints
Links:
- added link world
Joints:
- added joint base_to_ee_base_link: type fixed, parent world, child eef_base_link, origin xyz=0 0 0 rpy=0.0 0.0 0.0
- joint eef_base_to_tcp: origin xyz=0 0 0.185795 rpy=0.0 0.0 0.0 -> xyz=-0.002851003 0.001035 0.188155183 rpy=0.0 0.0 0.0
