Commit message: ECL robot model remake

File: src/coop_assembly/data/models/abb_irb4600_40_255/urdf/ECL_robot1_with_track.urdf (robot description, URDF)
Before this commit: robot abb_irb4600_40_255_track, 16 links, 15 joints
Links:
- link base_link: geometry collision mesh filename=package://abb_irb4600_40_255/meshes/collision/base_link.stl; visual mesh filename=package://abb_irb4600_40_255/meshes/visual/base_link.stl
- link eef_base_link: geometry collision mesh filename=../meshes/collision/princeton_gripper_collision_m.stl; visual mesh filename=../meshes/visual/princeton_gripper_visual_m.stl
- link linear_axis_base_link: geometry collision mesh filename=../meshes/collision/ecl_track_rail_1_collision_m.stl; visual mesh filename=../meshes/visual/ecl_track_rail_1_visual_m.stl
- link linear_axis_carriage: geometry collision mesh filename=../meshes/collision/ecl_track_carriage_1_collision_m.stl; visual mesh filename=../meshes/visual/ecl_track_carriage_1_visual_m.stl
- link link_1: geometry collision mesh filename=package://abb_irb4600_40_255/meshes/collision/link_1.stl; visual mesh filename=package://abb_irb4600_40_255/meshes/visual/link_1.stl
- link link_2: geometry collision mesh filename=package://abb_irb4600_40_255/meshes/collision/link_2.stl; visual mesh filename=package://abb_irb4600_40_255/meshes/visual/link_2.stl
- link link_3: geometry collision mesh filename=package://abb_irb4600_40_255/meshes/collision/link_3.stl; visual mesh filename=package://abb_irb4600_40_255/meshes/visual/link_3.stl
- link link_4: geometry collision mesh filename=package://abb_irb4600_40_255/meshes/collision/link_4.stl; visual mesh filename=package://abb_irb4600_40_255/meshes/visual/link_4.stl
- link link_5: geometry collision mesh filename=package://abb_irb4600_40_255/meshes/collision/link_5.stl; visual mesh filename=package://abb_irb4600_40_255/meshes/visual/link_5.stl
- link link_6: geometry collision mesh filename=package://abb_irb4600_40_255/meshes/collision/link_6.stl; visual mesh filename=package://abb_irb4600_40_255/meshes/visual/link_6.stl
Joints:
- joint linear_axis_actuation_joint: axis 1 0 0 -> 0 -1 0
- joint linear_axis_joint_1: origin xyz=-3.153 -0.212 0.470 rpy=0 0 0 -> xyz=0 0 0 rpy=0 0 0
- joint linear_axis_joint_3: origin xyz=0 0 0.470 rpy=0 0 0 -> xyz=0 0 0 rpy=0 0 0
- joint linear_axis_to_base_link: origin xyz=0 0 0 rpy=0 0 1.57079632679 -> xyz=0 0 0 rpy=0 0 0
- joint robot_to_linear_axis: origin xyz=0 0 0 rpy=0 0 -1.57079632679 -> xyz=0 0 0 rpy=0 0 0

Commit message: [WIP] test stream on abb_track

File: src/coop_assembly/data/models/abb_irb4600_40_255/urdf/ECL_robot1_with_track.urdf (robot description, URDF)
Before this commit: robot ECL_robot1_with_track, 16 links, 15 joints
Links:
- added link platform; collision mesh filename=../meshes/collision/floor_mounts_collision.stl
Joints:
- removed joint linear_axis_to_base_link
- added joint linear_axis_to_world_link: type fixed, parent world_link, child linear_axis_base_link, origin xyz=0 0 0 rpy=0 0 0
- added joint platform_to_world_link: type fixed, parent world_link, child platform, origin xyz=0 0 0 rpy=0 0 0
- joint eef_base_to_tcp: origin xyz=0.0 0.0 0.475 rpy=0 0 0 -> xyz=0.0 0.0 0.36 rpy=0 0 0
- joint linear_axis_actuation_joint: limit lower=0 upper=5.4 effort=1 velocity=1 -> lower=0 upper=3.6 effort=1 velocity=1

Commit message: abb_track stream verified

File: src/coop_assembly/data/models/abb_irb4600_40_255/urdf/ECL_robot1_with_track.urdf (robot description, URDF)
Before this commit: robot ECL_robot1_with_track, 17 links, 16 joints
Links:
- link base_link: geometry collision mesh filename=package://abb_irb4600_40_255/meshes/collision_pybullet/base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; visual mesh filename=package://abb_irb4600_40_255/meshes/visual/base_link.stl
- link link_1: geometry collision mesh filename=package://abb_irb4600_40_255/meshes/collision_pybullet/link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; visual mesh filename=package://abb_irb4600_40_255/meshes/visual/link_1.stl
- link link_2: geometry collision mesh filename=package://abb_irb4600_40_255/meshes/collision_pybullet/link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; visual mesh filename=package://abb_irb4600_40_255/meshes/visual/link_2.stl
- link link_3: geometry collision mesh filename=package://abb_irb4600_40_255/meshes/collision_pybullet/link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; visual mesh filename=package://abb_irb4600_40_255/meshes/visual/link_3.stl
- link link_4: geometry collision mesh filename=package://abb_irb4600_40_255/meshes/collision_pybullet/link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; visual mesh filename=package://abb_irb4600_40_255/meshes/visual/link_4.stl
- link link_5: geometry collision mesh filename=package://abb_irb4600_40_255/meshes/collision_pybullet/link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; visual mesh filename=package://abb_irb4600_40_255/meshes/visual/link_5.stl
- link link_6: geometry collision mesh filename=package://abb_irb4600_40_255/meshes/collision_pybullet/link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; visual mesh filename=package://abb_irb4600_40_255/meshes/visual/link_6.stl

Commit message: abb_track tet test working

File: src/coop_assembly/data/models/abb_irb4600_40_255/urdf/ECL_robot1_with_track.urdf (robot description, URDF)
Before this commit: robot ECL_robot1_with_track, 17 links, 16 joints
Links:
- removed link platform
Joints:
- removed joint platform_to_world_link

Commit message: abb track GH conf viz

File: src/coop_assembly/data/models/abb_irb4600_40_255/urdf/ECL_robot1_with_track.urdf (robot description, URDF)
Before this commit: robot ECL_robot1_with_track, 16 links, 15 joints
Links:
- link eef_base_link: geometry collision mesh filename=package://abb_irb4600_40_255/meshes/collision/princeton_gri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; visual mesh filename=package://abb_irb4600_40_255/meshes/visual/princeton_grippe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
- link linear_axis_base_link: geometry collision mesh filename=package://abb_irb4600_40_255/meshes/collision/ecl_track_rai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; visual mesh filename=package://abb_irb4600_40_255/meshes/visual/ecl_track_rail_1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
- link linear_axis_carriage: geometry collision mesh filename=package://abb_irb4600_40_255/meshes/collision/ecl_track_car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; visual mesh filename=package://abb_irb4600_40_255/meshes/visual/ecl_track_carria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
Joints:
- joint eef_base_to_tcp: origin xyz=0.0 0.0 0.36 rpy=0 0 0 -> xyz=0.0 0.0 0.3705 rpy=0 0 0
