Commit message: robotiq hand urdf get right

File: src/coop_assembly/data/models/robotiq_85/urdf/robotiq_85_gripper_simple.urdf (robot description, URDF)
Before this commit: robot robotiq_85_gripper, 16 links, 15 joints
Links:
- removed link base_link
- removed link dummy_center_indicator_link
- removed link pitch_control
- removed link roll_control
- removed link y_control
- removed link yaw_control
- removed link z_control
- added link bar_tcp
- added link robotiq_85_mount
Joints:
- removed joint center_x
- removed joint center_y
- removed joint center_z
- removed joint dummy_center_fixed_joint
- removed joint gripper_pitch
- removed joint gripper_roll
- removed joint gripper_yaw
- added joint mount: type fixed, parent robotiq_85_mount, child robotiq_85_base_link, origin xyz=0.0 0.0 0.0 rpy=0.0 -1.5707963267948966 1.5707963267948966
- added joint tool0-bar_tcp_fixed_joint: type fixed, parent robotiq_85_mount, child bar_tcp, origin xyz=0 0 0.138 rpy=0 0 3.141592653589793

File: src/coop_assembly/data/models/ur5e/urdf/ur5e.urdf (robot description, URDF)
Before this commit: robot ur5e, 11 links, 10 joints
Links:
- link base_link: geometry collision mesh filename=../meshes/collision/base.stl scale=1.0 1.0 1.0; visual mesh filename=../meshes/visual/base.dae
- link forearm_link: geometry collision mesh filename=../meshes/collision/forearm.stl scale=1.0 1.0 1.0; visual mesh filename=../meshes/visual/forearm.dae
- link shoulder_link: geometry collision mesh filename=../meshes/collision/shoulder.stl scale=1.0 1.0 1.0; visual mesh filename=../meshes/visual/shoulder.dae
- link upper_arm_link: geometry collision mesh filename=../meshes/collision/upperarm.stl scale=1.0 1.0 1.0; visual mesh filename=../meshes/visual/upperarm.dae
- link wrist_1_link: geometry collision mesh filename=../meshes/collision/wrist1.stl scale=1.0 1.0 1.0; visual mesh filename=../meshes/visual/wrist1.dae
- link wrist_2_link: geometry collision mesh filename=../meshes/collision/wrist2.stl scale=1.0 1.0 1.0; visual mesh filename=../meshes/visual/wrist2.dae
- link wrist_3_link: geometry collision mesh filename=../meshes/collision/wrist3.stl scale=1.0 1.0 1.0; visual mesh filename=../meshes/visual/wrist3.dae
